File: hardware/pacer.kicad_sch (KiCad schematic)
At the start: 38 parts, among them J1 Conn_01x04, J2 Conn_01x02_Pin, J3 Conn_01x02_Pin, J4 Conn_01x02_Socket, J5 Conn_01x02_Socket, SW1 SW_SPST, SW2 SW_SPDT, U1 CH32V003FxPx, U2 XCL103D333CR-G, U3 BU4210G-TR, U4 74HC595, U5 74HC595, U6 74HC595, Y1 Crystal_GND24

Commit message: PCB v1
Parts:
- removed BT1: Battery_Cell, Battery:BatteryHolder_Keystone_2460_1xAA, symbol Device:Battery_Cell
- removed D1, D2, D3, D4: LED, LED_SMD:LED_0603_1608Metric_Pad1.05x0.95mm_HandSolder, symbol Device:LED
- removed H3, H4: MountingHole, MountingHole:MountingHole_2.2mm_M2, symbol Mechanical:MountingHole
- removed J4, J5: Conn_01x02_Socket, Connector_PinSocket_2.54mm:PinSocket_1x02_P2.54mm_Vertical, symbol Connector:Conn_01x02_Socket
- removed LS1: PKM13EPYH4000-A0, My_lib:buzzer_pkm13, symbol Device:Speaker_Crystal
- removed SW1: SW_SPST, My_lib:DS-850K-S, symbol Switch:SW_SPST
- added BAR3: OSX05201-GGR1, My_lib:OSX05201-GGR1, symbol My_lib:OSX05201-GGR1
- added R3: 4.7k, Resistor_SMD:R_0603_1608Metric_Pad0.98x0.95mm_HandSolder, symbol Device:R
- renumbered SW2 to SW1
Connections:
- net +BATT: no longer J2.1 (Pin_1)
- net BUZZER: now also U1.1 (PD4); no longer U1.10 (PC0)
- net GND: now also U4.13 (~{OE}), U5.13 (~{OE}), U6.13 (~{OE}), BAR3.6 (K)
- net at RN6.1 (R1.1): now also BAR3.7 (K)
- net at RN6.2 (R2.1): now also BAR3.8 (K)
- net BUZZER_DRV: now reaches D5.1 (K), R2.2
- net BUZZER_DRV: now also J2.1 (Pin_1)
- net IND: now reaches U1.17 (PC7)
- net IND: now also R3.1
- net at SW1.1 (A): now also R2.1
- net at SW1.3 (C): no longer R2.1
- net at RN6.3 (R3.1): now also BAR3.9 (K)
- net at RN6.4 (R4.1): now also BAR3.10 (K)
- net IND1: no longer names the net of U4.3 (QD)
- net IND1: now also BAR3.1 (A)
- net IND2: no longer names the net of U4.2 (QC)
- net IND2: now also BAR3.2 (A)
- net IND3: no longer names the net of U4.1 (QB)
- net IND3: now also BAR3.3 (A)
- net IND4: no longer names the net of U4.15 (QA)
- net IND4: now also BAR3.4 (A)
- removed net ~{LED_OE}: U1.13 (PC3), U4.13 (~{OE}), U5.13 (~{OE}), U6.13 (~{OE})
- new net: BAR3.5 (A), R3.2
Other:
- note added: "+BATT"
- note added: "BUZZER_DRV"
- note added: "Battery, Buzzer"
- note added: "Bottom"
- note added: "GND"
- note added: "MCU, DCDC, LED, etc."
- note added: "Top"
- moved on the sheet: BAR1, BAR2, D5, J2, J3, R2, RN1, RN2, RN3, RN4, RN5, RN6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

Commit message: jlcpcb production files
Parts:
- BAR1, BAR2, BAR3, J1, J2, J3, SW1: now left out of the parts list
- R2: value 1k -> 1.2k
- R3: value 4.7k -> 5.6k
- RN6: value 4.7k -> 1k
Changed lines of the file:
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@@
 		(unit 1)
 		(exclude_from_sim no)
-		(in_bom yes)
+		(in_bom no)
 		(on_board yes)
 		(dnp no)
@@
 		(unit 1)
 		(exclude_from_sim no)
-		(in_bom yes)
+		(in_bom no)
 		(on_board yes)
 		(dnp no)
@@
 		(unit 1)
 		(exclude_from_sim no)
-		(in_bom yes)
+		(in_bom no)
 		(on_board yes)
 		(dnp no)
@@
 		(unit 1)
 		(exclude_from_sim no)
-		(in_bom yes)
+		(in_bom no)
 		(on_board yes)
 		(dnp no)
@@
 		(unit 1)
 		(exclude_from_sim no)
-		(in_bom yes)
+		(in_bom no)
 		(on_board yes)
 		(dnp no)
@@
 		(unit 1)
 		(exclude_from_sim no)
-		(in_bom yes)
+		(in_bom no)
 		(on_board yes)
 		(dnp no)
@@
 			)
 		)
-		(property "Value" "4.7k"
+		(property "Value" "1k"
 			(at 198.12 27.94 90)
 			(effects
@@
 		(unit 1)
 		(exclude_from_sim no)
-		(in_bom yes)
+		(in_bom no)
 		(on_board yes)
 		(dnp no)
@@
 			)
 		)
-		(property "Value" "1k"
+		(property "Value" "1.2k"
 			(at 55.88 149.86 90)
 			(effects
@@
 			)
 		)
-		(property "Value" "4.7k"
+		(property "Value" "5.6k"
 			(at 163.83 25.4 90)
 			(effects

Commit message: add capacitors
Parts:
- added C10, C8, C9: 0.1u, Capacitor_SMD:C_0402_1005Metric_Pad0.74x0.62mm_HandSolder, symbol Device:C
- added C6: 100p, Capacitor_SMD:C_0402_1005Metric_Pad0.74x0.62mm_HandSolder, symbol Device:C
- added C7: 1n, Capacitor_SMD:C_0402_1005Metric_Pad0.74x0.62mm_HandSolder, symbol Device:C
Connections:
- net +3V3: now also C10.1, C8.1, C9.1
- net GND: now also C10.2, C6.2, C7.2, C8.2, C9.2
- net at R1.2, U2.3 (CE), U3.1 (VOUT): now also C7.1
- net at U3.5 (CT): now also C6.1
- no-connect marks 12 -> 11
Other:
- moved on the sheet: BAR1, BAR2, BAR3, J2, J3, R1, R3, RN1, RN2, RN3, RN4, RN5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
