File: hardware/pacer.kicad_pcb (KiCad board)
At the start: 2 copper layers, 63.4 x 28.1 mm, 35 parts, among them J1 Conn_01x04, J2 Conn_01x02_Pin, J3 Conn_01x02_Pin, SW1 SW_SPDT, U1 CH32V003FxPx, U2 XCL103D333CR-G, U3 BU4210G-TR, U4 74HC595, U5 74HC595, U6 74HC595, Y1 Crystal_GND24

Commit message: minor PCB fix
Parts:
- moved C10 12.9 mm to (90.1, 109.1), turned to 90 degrees
- moved J3 2.54 mm to (146.6, 112.3), turned to 0 degrees
Routing:
- net +3V3: track 160.9 -> 165.6 mm
- net GND: track 220.7 -> 221.8 mm
