File: hardware/pacer_bottom/pacer_bottom.kicad_pcb (KiCad board)
At the start: 2 copper layers, 88.2 x 28.1 mm, 11 parts, among them J1 Conn_01x02_Socket, J2 Conn_01x02_Socket, SW1 SW_SPST

Commit message: update silkscreen
Parts:
- added G***: LOGO, LOGO, B.Cu at (166.6, 88.7)
- added G***: LOGO, LOGO, B.Cu at (180.3, 93.8)
- moved G*** 57.4 mm to (110.7, 100.0)
Other:
- board text added: "Pacer designed by object1037"
- board text removed: "AA Battery"
