File: hardware/pacer_bottom/pacer_bottom.kicad_sch (KiCad schematic)
At the start: 10 parts, among them J1 Conn_01x02_Socket, J2 Conn_01x02_Socket, SW1 SW_SPST

Commit message: hardware update after prototype
Parts:
- removed H1, H2: MountingHole, My_lib:OSX10201-mount, symbol Mechanical:MountingHole
- removed H3: MountingHole, My_lib:OSX05201-mount, symbol Mechanical:MountingHole
- renumbered H4 to H1, H5 to H2
Other:
- moved on the sheet: H1, H2
